Commit message: removed imu

File: robots/aliengo_description/xacro/gazebo.xacro (robot description, xacro)
@@ -36,5 +36,5 @@
         </plugin>
     </gazebo>
-    <gazebo reference="imu_link">
+    <!-- <gazebo reference="imu_link">
         <gravity>true</gravity>
         <sensor name="imu_sensor" type="imu">
@@ -54,5 +54,5 @@
             <pose>0 0 0 0 0 0</pose>
         </sensor>
-    </gazebo>
+    </gazebo> -->
     <!-- Foot contacts. -->
     <gazebo reference="FR_calf">

File: robots/aliengo_description/xacro/robot.xacro (robot description, xacro)
@@ -87,5 +87,5 @@
         </link>
     </xacro:if>
-    <joint name="imu_joint" type="fixed">
+    <!-- <joint name="imu_joint" type="fixed">
         <parent link="trunk"/>
         <child link="imu_link"/>
@@ -111,5 +111,5 @@
             </geometry>
         </collision>
-    </link>
+    </link> -->
     <xacro:leg name="FR" mirror="-1" mirror_dae= "False" front_hind="1" front_hind_dae="True">
         <origin rpy="0 0 0" xyz="${leg_offset_x} ${-leg_offset_y} 0"/>
