Commit message: added accessories for nav

File: robots/aliengo_description/xacro/aliengo.champ.urdf (robot description, URDF)
Before this commit: robot aliengo_description, 18 links, 17 joints
Links:
- added link camera_depth_frame
- added link camera_depth_optical_frame
- added link camera_link, mass 0.200; collision mesh filename=package://hector_sensors_description/meshes/asus_camera/asu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; visual mesh filename=package://hector_sensors_description/meshes/asus_camera/asu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
- added link camera_rgb_frame
- added link camera_rgb_optical_frame
- added link hokuyo_frame, mass 0.270; collision box size=0.058 0.058 0.087; visual mesh filename=package://hector_sensors_description/meshes/hokuyo_utm30lx/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
- added link imu_link, mass 0.001
Joints:
- added joint camera_depth_joint: type fixed, parent camera_link, child camera_depth_frame, origin xyz=0.0 0.049 0.0 rpy=0 0 0
- added joint camera_depth_optical_joint: type fixed, parent camera_depth_frame, child camera_depth_optical_frame, origin xyz=0 0 0 rpy=-1.57079632679 0.0 -1.57079632679
- added joint camera_joint: type fixed, parent trunk, child camera_link, origin xyz=0.3235 0.0 -0.066 rpy=0 0 0
- added joint camera_rgb_joint: type fixed, parent camera_link, child camera_rgb_frame, origin xyz=0.0 0.022 0.0 rpy=0 0 0
- added joint camera_rgb_optical_joint: type fixed, parent camera_rgb_frame, child camera_rgb_optical_frame, origin xyz=0 0 0 rpy=-1.57079632679 0.0 -1.57079632679
- added joint hokuyo_joint: type fixed, parent trunk, child hokuyo_frame, origin xyz=0.0 0.0 0.096 rpy=0 0 0
- added joint imu_joint: type fixed, parent trunk, child imu_link

File: robots/aliengo_description/xacro/robot.xacro (robot description, xacro)
@@ -125,3 +125,9 @@
     </xacro:leg>
     <!-- <xacro:stairs stairs="15" xpos="0" ypos="2.0" zpos="0" /> -->
+    <xacro:include filename="$(find champ_description)/urdf/accessories.urdf.xacro" />
+    <xacro:accessories
+        base_name="trunk"
+        base_length="${trunk_length}"
+        base_height="${trunk_height}"
+    />
 </robot>
