Commit message: add hokuyo lidar to go1

File: robots/go1_description/xacro/go1.champ.urdf (robot description, URDF)
Before this commit: robot go1_description, 38 links, 37 joints
Links:
- added link hokuyo_frame, mass 0.270; collision box size=0.058 0.058 0.087; visual mesh filename=package://hector_sensors_description/meshes/hokuyo_utm30lx/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
Joints:
- added joint hokuyo_joint: type fixed, parent base, child hokuyo_frame, origin xyz=0.0 0.0 0.105 rpy=0 0 0

Commit message: rotate face_camera 180 deg

File: robots/go1_description/xacro/go1.champ.urdf (robot description, URDF)
Before this commit: robot go1_description, 39 links, 38 joints
Joints:
- joint camera_joint_face: origin xyz=0.2785 0.0125 0.0167 rpy=3.141592653589793 0 0 -> xyz=0.2785 0.0125 0.0167 rpy=0 0 0

Commit message: hokuyo_frame is on trunk, not base

File: robots/go1_description/xacro/go1.champ.urdf (robot description, URDF)
Before this commit: robot go1_description, 39 links, 38 joints
Joints:
- joint hokuyo_joint: parent base -> trunk
